File: PCB/nes-cartridge.sch (EAGLE design)
At the start: 17 parts, among them U1 ATtiny13A, U2 FLASH 512K x 8, U3 FLASH 512K x 8

Commit message: Cart board and programmer board checkpoint.
Parts:
- removed PA132EDGE, PA142EDGE: (no value), rlc:SOLDER_JUMPER-80MIL-RND
- removed R2, R3: 10K, rlc:RESISTOR0603
- renumbered PRG!W!_2EDGE to PRG-WREN, U2 to CHR-MEM, U3 to PRG-MEM
Connections:
- removed net PPU_A13: CHR-MEM.A13, PA132EDGE.P$2, R3.1
- removed net PPU_A13EDGE: PA132EDGE.P$1, PCB1.EXP6
- removed net PPU_A14: CHR-MEM.A14, PA142EDGE.P$2, R2.1
- removed net PPU_A14EDGE: PA142EDGE.P$1, PCB1.EXP5
- net GND: now also CHR-MEM.A13, CHR-MEM.A14, CHR-MEM.A15, CHR-MEM.A16, CHR-MEM.A17, CHR-MEM.A18, PRG-MEM.A15, PRG-MEM.A16, PRG-MEM.A17, PRG-MEM.A18
- net VCC: no longer R2.2, R3.2
Other:
- note added: "CHR WREN?"
- note added: "Special thanks to ViGrey: https://vigrey.com/nes NES DEV Wiki https://www.nesdev.org/wiki/Nesdev_Wiki"
- note removed: "Special thanks to ViGrey: https://vigrey.com/nes"
