File: PCB/nes-cartridge.brd (EAGLE design)
At the start: 100 x 40 mm, 17 parts, among them U1 ATtiny13A, U2 FLASH 512K x 8, U3 FLASH 512K x 8

Commit message: Cart board and programmer board checkpoint.
Parts:
- removed PA132EDGE, PA142EDGE: (no value), rlc:SOLDER_JUMP_80MIL_RND
- removed R2, R3: 10K, rlc:0603-RES
- moved R1 6.00 mm to (45.0, 30.0)
- moved H_SCROLL 3.00 mm to (50.0, 24.0)
- moved V_SCROLL 3.00 mm to (50.0, 28.0)
- renumbered PRG!W!_2EDGE to PRG-WREN, U2 to CHR-MEM, U3 to PRG-MEM
Connections:
- removed net PPU_A13: CHR-MEM.4, PA132EDGE.2, R3.1
- removed net PPU_A13EDGE: PA132EDGE.1, PCB1.54
- removed net PPU_A14: CHR-MEM.5, PA142EDGE.2, R2.1
- removed net PPU_A14EDGE: PA142EDGE.1, PCB1.55
- net GND: now also CHR-MEM.10, CHR-MEM.11, CHR-MEM.4, CHR-MEM.5, CHR-MEM.6, CHR-MEM.9, PRG-MEM.10, PRG-MEM.11, PRG-MEM.6, PRG-MEM.9
- net VCC: no longer R2.2, R3.2
Routing:
- net PPU_A13: track 32.2 -> 0.00 mm, vias 2 -> 0
- net PPU_A14: track 30.7 -> 0.00 mm, vias 3 -> 0
- net PPU_!WR: track 47.9 -> 35.4 mm, vias 2 -> 3
- net PPU_A14EDGE: track 11.0 -> 0.00 mm, vias 1 -> 0
- net PPU_A13EDGE: track 9.88 -> 0.00 mm, vias 1 -> 0
- net CIRAM_A10: track 25.0 -> 28.8 mm
- net VCC: track 120.6 -> 116.9 mm
- net PPU_A10: track 48.3 -> 50.7 mm
- net PPU_A11: track 39.6 -> 41.7 mm
- net CPU_D5: track 33.7 -> 34.9 mm
- net CPU_A5: track 33.3 -> 34.3 mm
- net CPU_A13: track 29.7 -> 29.0 mm
- net GND: vias 31 -> 60
Other:
- outline, holes or cut-outs redrawn
- board text added: "2023-12"
- board text added: "CircuitMonkey"
- board text added: "MNEMOSYNE-1"
- board text added: "NES Flash Cartidge"
- board text added: "Rev. A"

Commit message: Final tweaks.
Routing:
- net PPU_A10: track 50.7 -> 52.2 mm
- net CIC_!RST: track 65.8 -> 66.8 mm
- net PPU_D3: track 28.1 -> 28.8 mm
- net PPU_D2: track 29.4 -> 29.9 mm
